Commit message: modify wrist amount glb color

File: mani_skill/assets/robots/panda/panda_irom.urdf (robot description, URDF)
Before this commit: robot panda, 17 links, 16 joints
Links:
- link camera_link: geometry collision mesh filename=realsense2_description/meshes/wrist_mount_irom.glb; visual mesh filename=realsense2_description/meshes/wrist_mount_irom.glb
Joints:
- joint panda_hand_tcp_joint: origin xyz=0 0 0.175 rpy=0 0 0 -> xyz=0 0 0 rpy=0 0 0

Commit message: Add visually more similar gripper glb

File: mani_skill/assets/robots/panda/panda_irom.urdf (robot description, URDF)
Before this commit: robot panda, 17 links, 16 joints
Links:
- link camera_link: geometry collision mesh filename=realsense2_description/meshes/wrist_mount_irom.stl; visual mesh filename=realsense2_description/meshes/wrist_mount_irom.glb
Joints:
- joint camera_reference_joint: origin xyz=0.02 0 0 rpy=3.1415926 0 0  -> xyz=0.0 0 0 rpy=3.1415926 0 0 

Commit message: modify wrist mount meshes

File: mani_skill/assets/robots/panda/panda_irom.urdf (robot description, URDF)
Before this commit: robot panda, 17 links, 16 joints
Links:
- removed link camera_reference_link
- removed link camera_reference_link_flipped
Joints:
- removed joint camera_reference_joint
- removed joint camera_reference_joint_flipped

Commit message: modify panda urdf

File: mani_skill/assets/robots/panda/panda_irom.urdf (robot description, URDF)
Before this commit: robot panda, 15 links, 14 joints
Joints:
- joint panda_hand_tcp_joint: origin xyz=0 0 0 rpy=0 0 0 -> xyz=0 0 0.21 rpy=0 0 0
